File: eagle/Display.brd (EAGLE design)
At the start: 94 x 40.3 mm, 34 parts

Commit message: Updated schematics
Connections:
- net S$7: no longer E$16.1
- net S$8: now also E$16.1
Routing:
- net S$8: track 64.8 -> 87.8 mm, vias 0 -> 1
- net S$6: track 92.3 -> 87.3 mm
- net S$7: track 76.6 -> 80.8 mm
Changed lines of the file:
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@@
 <?xml version="1.0" encoding="utf-8"?>
 <!DOCTYPE eagle SYSTEM "eagle.dtd">
-<eagle version="6.1">
+<eagle version="6.5.0">
 <drawing>
 <settings>
@@
 </class>
 </classes>
-<designrules>
+<designrules name="default">
 <description language="en">&lt;b&gt;EAGLE Design Rules&lt;/b&gt;
 &lt;p&gt;
@@
 <wire x1="27.94" y1="22.86" x2="5.08" y2="22.86" width="0.6096" layer="16"/>
 <wire x1="27.94" y1="22.86" x2="50.8" y2="22.86" width="0.6096" layer="16"/>
-<wire x1="69.85" y1="22.86" x2="73.66" y2="22.86" width="0.6096" layer="16"/>
-<wire x1="68.58" y1="21.59" x2="69.85" y2="22.86" width="0.6096" layer="16"/>
-<wire x1="53.34" y1="21.59" x2="68.58" y2="21.59" width="0.6096" layer="16"/>
+<wire x1="71.12" y1="22.86" x2="73.66" y2="22.86" width="0.6096" layer="16"/>
+<wire x1="69.85" y1="21.59" x2="71.12" y2="22.86" width="0.6096" layer="16"/>
+<wire x1="53.34" y1="21.59" x2="69.85" y2="21.59" width="0.6096" layer="16"/>
 <wire x1="52.07" y1="22.86" x2="53.34" y2="21.59" width="0.6096" layer="16"/>
 <wire x1="50.8" y1="22.86" x2="52.07" y2="22.86" width="0.6096" layer="16"/>
@@
 <wire x1="27.94" y1="20.32" x2="26.67" y2="20.32" width="0.6096" layer="16"/>
 <wire x1="52.07" y1="12.7" x2="55.88" y2="8.89" width="0.6096" layer="1"/>
-<wire x1="57.15" y1="12.7" x2="52.07" y2="12.7" width="0.6096" layer="16"/>
-<wire x1="64.77" y1="20.32" x2="57.15" y2="12.7" width="0.6096" layer="16"/>
-<wire x1="73.66" y1="20.32" x2="64.77" y2="20.32" width="0.6096" layer="16"/>
+<wire x1="59.69" y1="20.32" x2="52.07" y2="12.7" width="0.6096" layer="16"/>
+<wire x1="73.66" y1="20.32" x2="59.69" y2="20.32" width="0.6096" layer="16"/>
 <wire x1="55.88" y1="8.89" x2="55.88" y2="8.47" width="0.6096" layer="1"/>
-<wire x1="64.77" y1="20.32" x2="50.8" y2="20.32" width="0.6096" layer="16"/>
+<wire x1="59.69" y1="20.32" x2="50.8" y2="20.32" width="0.6096" layer="16"/>
 <wire x1="33.02" y1="20.32" x2="27.94" y2="20.32" width="0.6096" layer="16"/>
 <wire x1="34.29" y1="21.59" x2="33.02" y2="20.32" width="0.6096" layer="16"/>
@@
 <contactref element="E$9" pad="1"/>
 <contactref element="E$13" pad="1"/>
-<contactref element="E$16" pad="1"/>
 <contactref element="E$5" pad="1"/>
 <contactref element="E$1" pad="1"/>
@@
 <wire x1="60.96" y1="10.16" x2="60.96" y2="8.47" width="0.6096" layer="1"/>
 <wire x1="66.04" y1="15.24" x2="60.96" y2="10.16" width="0.6096" layer="16"/>
-<wire x1="66.04" y1="15.24" x2="73.66" y2="15.24" width="0.6096" layer="16"/>
-<wire x1="73.66" y1="15.24" x2="88.9" y2="15.24" width="0.6096" layer="16"/>
 <wire x1="48.26" y1="10.16" x2="43.18" y2="15.24" width="0.6096" layer="1"/>
 <wire x1="60.96" y1="10.16" x2="48.26" y2="10.16" width="0.6096" layer="16"/>
 <via x="60.96" y="10.16" extent="1-16" drill="0.508"/>
 <via x="48.26" y="10.16" extent="1-16" drill="0.508"/>
+<wire x1="66.04" y1="15.24" x2="67.31" y2="15.24" width="0.6096" layer="16"/>
+<wire x1="67.31" y1="15.24" x2="72.39" y2="10.16" width="0.6096" layer="16"/>
+<wire x1="72.39" y1="10.16" x2="83.82" y2="10.16" width="0.6096" layer="16"/>
+<wire x1="83.82" y1="10.16" x2="88.9" y2="15.24" width="0.6096" layer="16"/>
 </signal>
 <signal name="S$8">
@@
 <contactref element="E$4" pad="1"/>
 <contactref element="E$22" pad="2"/>
-<wire x1="52.07" y1="15.24" x2="58.42" y2="8.89" width="0.6096" layer="1"/>
-<wire x1="50.8" y1="15.24" x2="52.07" y2="15.24" width="0.6096" layer="1"/>
+<wire x1="57.15" y1="15.24" x2="57.785" y2="15.24" width="0.6096" layer="1"/>
+<wire x1="57.785" y1="15.24" x2="57.785" y2="9.525" width="0.6096" layer="1"/>
+<wire x1="57.785" y1="9.525" x2="58.42" y2="8.89" width="0.6096" layer="1"/>
 <wire x1="58.42" y1="8.89" x2="58.42" y2="8.47" width="0.6096" layer="1"/>
 <wire x1="11.43" y1="15.24" x2="5.08" y2="15.24" width="0.6096" layer="1"/>
@@
 <wire x1="29.21" y1="15.24" x2="34.29" y2="20.32" width="0.6096" layer="16"/>
 <wire x1="27.94" y1="15.24" x2="29.21" y2="15.24" width="0.6096" layer="16"/>
+<contactref element="E$16" pad="1"/>
+<wire x1="50.8" y1="15.24" x2="57.15" y2="15.24" width="0.6096" layer="1"/>
+<via x="57.15" y="15.24" extent="1-16" drill="0.6"/>
+<wire x1="57.15" y1="15.24" x2="60.96" y2="19.05" width="0.6096" layer="16"/>
+<wire x1="60.96" y1="19.05" x2="68.58" y2="19.05" width="0.6096" layer="16"/>
+<wire x1="68.58" y1="19.05" x2="72.39" y2="15.24" width="0.6096" layer="16"/>
+<wire x1="72.39" y1="15.24" x2="73.66" y2="15.24" width="0.6096" layer="16"/>
 </signal>
 <signal name="S$9">
